File: hardware/PCB/THT/SedNav_Windsensor_THT.kicad_sch (KiCad schematic)
At the start: 11 parts, among them IC1 AS5600-ASOT, J1 Conn_01x02_Pin, U1 XIAO-ESP32-C6, U2 StpDwnE3.3-0.5, U3 SS411P, U4 DS18B20

Commit message: Changed connector
Parts:
- J1: footprint Connector_JST:JST_XH_B2B-XH-A_1x02_P2.50mm_Vertical -> Connector_JST:JST_ZH_B2B-ZR_1x02_P1.50mm_Vertical
Changed lines of the file:
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@@
 			)
 		)
-		(property "Footprint" "Connector_JST:JST_XH_B2B-XH-A_1x02_P2.50mm_Vertical"
+		(property "Footprint" "Connector_JST:JST_ZH_B2B-ZR_1x02_P1.50mm_Vertical"
 			(at 44.45 68.58 0)
 			(effects

Commit message: V3.1 du PCB THT
Parts:
- J1: footprint Connector_JST:JST_ZH_B2B-ZR_1x02_P1.50mm_Vertical -> TerminalBlock_Phoenix:TerminalBlock_Phoenix_MPT-0,5-2-2.54_1x02_P2.54mm_Horizontal
Changed lines of the file:
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@@
 			)
 		)
-		(property "Footprint" "Connector_JST:JST_ZH_B2B-ZR_1x02_P1.50mm_Vertical"
+		(property "Footprint" "TerminalBlock_Phoenix:TerminalBlock_Phoenix_MPT-0,5-2-2.54_1x02_P2.54mm_Horizontal"
 			(at 44.45 68.58 0)
 			(effects
@@
 			)
 		)
-		(property "Datasheet" "https://www.recom-power.com/pdf/Innoline/R-78Exx-0.5.pdf"
+		(property "Datasheet" "https://recom-power.com/pdf/Innoline/R-78K-0.5.pdf"
 			(at 80.01 68.58 0)
 			(effects
@@
 			)
 		)
-		(property "Description" "500mA Step-Down DC/DC-Regulator, 6-28V input, 3.3V fixed Output Voltage, LM78xx replacement, -40°C to +85°C, SIP3"
+		(property "Description" "500mA Step-Down DC/DC-Regulator, 4.5-36V input, 3.3V fixed Output Voltage, LM78xx replacement, -40°C to +90°C, SIP3"
 			(at 80.01 68.58 0)
 			(effects
