File: hardware/PCB/THT/SedNav_Windsensor_THT.kicad_pcb (KiCad board)
At the start: 2 copper layers, 33 x 33 mm, 14 parts, among them IC1 AS5600-ASOT, J1 Conn_01x02_Pin, M2_1 MountingHole_2.2mm_M2_Pad_Top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, M2_2 MountingHole_2.2mm_M2_Pad_Top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, U1 XIAO-ESP32-C6, U2 StpDwnE3.3-0.5, U3 SS411P, U4 DS18B20

Commit message: Changed connector
Parts:
- J1: footprint Connector_JST:JST_XH_B2B-XH-A_1x02_P2.50mm_Vertical -> Connector_JST:JST_ZH_B2B-ZR_1x02_P1.50mm_Vertical; moved to B.Cu
- moved J1 4.28 mm to (121.2, 61.0), turned to 60 degrees
Routing:
- net VCC: track 12.6 -> 6.70 mm
Other:
- board text added: "+"
- board text added: "-"
- board text added: "SedNav Windsensor THT v3"
- board text removed: "GND"
- board text removed: "SedNav Windsensor THT v2"
- board text removed: "VCC"

Commit message: V3.1 du PCB THT
Parts:
- J1: footprint Connector_JST:JST_ZH_B2B-ZR_1x02_P1.50mm_Vertical -> TerminalBlock_Phoenix:TerminalBlock_Phoenix_MPT-0,5-2-2.54_1x02_P2.54mm_Horizontal
- moved D1 5.45 mm to (124.1, 69.1), turned to 120 degrees
- moved J1 3.82 mm to (121.5, 57.2), turned to 180 degrees
- moved U2 1.10 mm to (127.9, 65.3)
Routing:
- net +3.3V: track 76.0 -> 73.0 mm
- net Net-(D1-K): track 3.95 -> 5.51 mm
- net VCC: track 6.70 -> 5.79 mm
Other:
- board text added: "4.5 to 36VDC"
- board text added: "SedNav Windsensor THT v3.1"
- board text removed: "4.5-36VDC"
- board text removed: "SedNav Windsensor THT v3"

Commit message: Version finale, fin du projet
Other:
- board text added: "4.5 to 36V"
- board text removed: "4.5 to 36VDC"
Changed lines of the file:
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@@
 			)
 		)
+		(property "MPN" "SS411P"
+			(at 0 0 0)
+			(unlocked yes)
+			(layer "F.Fab")
+			(hide yes)
+			(effects
+				(font
+					(size 1 1)
+					(thickness 0.15)
+				)
+			)
+		)
 		(property ki_fp_filters "TO-92*")
 		(sheetname "/")
@@
 			)
 		)
+		(property "MPN" "DS18B20+"
+			(at 0 0 0)
+			(unlocked yes)
+			(layer "F.Fab")
+			(hide yes)
+			(effects
+				(font
+					(size 1 1)
+					(thickness 0.15)
+				)
+			)
+		)
 		(property ki_fp_filters "TO*92*")
 		(sheetname "/")
@@
 			)
 		)
-		(property "Description" ""
+		(property "Description" "Microcontrôleur avec wifi intégré"
 			(at -0.045 0 90)
 			(unlocked yes)
@@
 			)
 		)
-		(property "Notes" "D'abord placer les résistances et le condensateur en dessous !"
+		(property "Notes" "D'abord placer les résistances et le condensateur en dessous, en faisant attention à ce que leurs pattes ne touchent pas le dessous de l'ESP32. Il faut couper le pin D6 qui n'est pas utilisé, afin de permettre l'installation du convertisseur de tension."
 			(at 0 0 0)
 			(unlocked yes)
@@
 			)
 		)
+		(property "MPN" "SB160"
+			(at 0 0 0)
+			(unlocked yes)
+			(layer "F.Fab")
+			(hide yes)
+			(effects
+				(font
+					(size 1 1)
+					(thickness 0.15)
+				)
+			)
+		)
 		(property ki_fp_filters "D*DO?41*")
 		(sheetname "/")
@@
 			)
 		)
+		(property "MPN" "AS5600-ASOT"
+			(at 0 0 0)
+			(unlocked yes)
+			(layer "B.Fab")
+			(hide yes)
+			(effects
+				(font
+					(size 1 1)
+					(thickness 0.15)
+				)
+				(justify mirror)
+			)
+		)
 		(sheetname "/")
 		(sheetfile "SedNav_Windsensor_THT.kicad_sch")
@@
 			)
 		)
+		(property "MPN" "RN55D4701FRE6"
+			(at 0 0 0)
+			(unlocked yes)
+			(layer "B.Fab")
+			(hide yes)
+			(effects
+				(font
+					(size 1 1)
+					(thickness 0.15)
+				)
+				(justify mirror)
+			)
+		)
 		(property ki_fp_filters "R_*")
 		(sheetname "/")
@@
 			)
 		)
+		(property "MPN" "MKP1837410161G"
+			(at 0 0 0)
+			(unlocked yes)
+			(layer "B.Fab")
+			(hide yes)
+			(effects
+				(font
+					(size 1 1)
+					(thickness 0.15)
+				)
+				(justify mirror)
+			)
+		)
 		(property ki_fp_filters "C_*")
 		(sheetname "/")
@@
 			)
 		)
+		(property "MPN" "RN55D4701FRE6"
+			(at 0 0 0)
+			(unlocked yes)
+			(layer "B.Fab")
+			(hide yes)
+			(effects
+				(font
+					(size 1 1)
+					(thickness 0.15)
+				)
+				(justify mirror)
+			)
+		)
 		(property ki_fp_filters "R_*")
 		(sheetname "/")
@@
 			)
 		)
+		(property "MPN" "R-78E3.3-0.5"
+			(at 0 0 0)
+			(unlocked yes)
+			(layer "B.Fab")
+			(hide yes)
+			(effects
+				(font
+					(size 1 1)
+					(thickness 0.15)
+				)
+				(justify mirror)
+			)
+		)
 		(property ki_fp_filters "Converter*DCDC*RECOM*R*78E*0.5*")
 		(sheetname "/")
@@
 			)
 		)
+		(property "MPN" "MPT 0.5/ 2-2.54"
+			(at 0 0 0)
+			(unlocked yes)
+			(layer "B.Fab")
+			(hide yes)
+			(effects
+				(font
+					(size 1 1)
+					(thickness 0.15)
+				)
+				(justify mirror)
+			)
+		)
 		(property ki_fp_filters "Connector*:*_1x??_*")
 		(sheetname "/")
@@
 		(fp_line
 			(start 4.16 -3.22)
+			(end 3.57 -3.22)
+			(stroke
+				(width 0.12)
+				(type solid)
+			)
+			(layer "B.SilkS")
+		)
+		(fp_line
+			(start 3.57 -2.6)
+			(end 4.16 -2.6)
+			(stroke
+				(width 0.12)
+				(type solid)
+			)
+			(layer "B.SilkS")
+		)
+		(fp_line
+			(start 1.51 -3.22)
+			(end 1.03 -3.22)
+			(stroke
+				(width 0.12)
+				(type solid)
+			)
+			(layer "B.SilkS")
+		)
+		(fp_line
+			(start 1.03 -2.6)
+			(end 1.51 -2.6)
+			(stroke
+				(width 0.12)
+				(type solid)
+			)
+			(layer "B.SilkS")
+		)
+		(fp_line
+			(start -1.03 -3.22)
 			(end -1.62 -3.22)
 			(stroke
@@
 		(fp_line
 			(start -1.62 -2.6)
-			(end 4.16 -2.6)
+			(end -1.03 -2.6)
 			(stroke
 				(width 0.12)
@@
 			(layer "B.SilkS")
 		)
-		(fp_poly
-			(pts
-				(xy -2 3.6) (xy 4.539999 3.6) (xy 4.54 -3.599999) (xy -2 -3.6)
-			)
+		(fp_rect
+			(start -2 3.6)
+			(end 4.54 -3.6)
 			(stroke
 				(width 0.05)
@@
 		(fp_line
 			(start -1.5 2.7)
-			(end 4.040001 2.7)
+			(end 4.04 2.7)
 			(stroke
 				(width 0.1)
@@
 			)
 		)
+		(pad "" np_thru_hole circle
+			(at 0 -2.54 180)
+			(size 1.1 1.1)
+			(drill 1.1)
+			(layers "*.Cu" "*.Mask")
+		)
+		(pad "" np_thru_hole circle
+			(at 2.54 -2.54 180)
+			(size 1.1 1.1)
+			(drill 1.1)
+			(layers "*.Cu" "*.Mask")
+		)
 		(pad "1" thru_hole roundrect
 			(at 0 0 180)
-			(size 2.1 2.2)
+			(size 2.2 2.2)
 			(drill 1.1)
 			(layers "*.Cu" "*.Mask")
@@
 		(pad "2" thru_hole circle
 			(at 2.54 0 180)
-			(size 2.1 2.1)
+			(size 2.2 2.2)
 			(drill 1.1)
 			(layers "*.Cu" "*.Mask")
@@
 			)
 		)
+		(property "MPN" "RN55D4701FRE6"
+			(at 0 0 0)
+			(unlocked yes)
+			(layer "B.Fab")
+			(hide yes)
+			(effects
+				(font
+					(size 1 1)
+					(thickness 0.15)
+				)
+				(justify mirror)
+			)
+		)
 		(property ki_fp_filters "R_*")
 		(sheetname "/")
@@
 		)
 	)
-	(gr_text "4.5\nto\n36VDC"
-		(at 117.715 58.25 270)
+	(gr_text "4.5\nto\n36V"
+		(at 117.965 56 270)
 		(layer "F.SilkS")
 		(effects
@@
 				(thickness 0.1)
 			)
-			(justify left bottom)
+			(justify right bottom)
 		)
 	)
@@
 	)
 	(zone
-		(net 1)
-		(net_name "+3.3V")
+		(net 16)
+		(net_name "Net-(D1-K)")
 		(layer "F.Cu")
 		(name "$teardrop_padvia$")
 		(hatch none 0.1)
-		(priority 30000)
+		(priority 30001)
 		(attr
 			(teardrop
@@
 		(polygon
 			(pts
-				(xy 125.739667 64.244905) (xy 125.631944 64.345815) (xy 125.532684 64.425672) (xy 125.441785 64.48672)
-				(xy 125.35599 64.533467) (xy 125.181232 64.59972) (xy 125.036344 64.636715) (xy 124.899079 64.671204)
-				(xy 124.748658 64.720228) (xy 124.578483 64.796762) (xy 124.381951 64.913786) (xy 124.827089 65.581747)
-				(xy 125.49505 66.026885) (xy 125.572904 65.901874) (xy 125.633378 65.787906) (xy 125.718607 65.573966)
-				(xy 125.77212 65.372492) (xy 125.813655 65.212341) (xy 125.876819 65.049865) (xy 125.924004 64.963946)
-				(xy 125.985587 64.872872) (xy 126.064564 64.775121) (xy 126.163931 64.669169)
+				(xy 127.99903 68.799115) (xy 127.99903 69.399115) (xy 129.299821 69.08961) (xy 129.228206 68.121039)
+				(xy 128.130971 68.414774)
 			)
 		)
 	)
 	(zone
-		(net 16)
-		(net_name "Net-(D1-K)")
+		(net 1)
+		(net_name "+3.3V")
 		(layer "F.Cu")
 		(name "$teardrop_padvia$")
 		(hatch none 0.1)
-		(priority 30001)
+		(priority 30000)
 		(attr
 			(teardrop
@@
 		(polygon
 			(pts
-				(xy 127.99903 68.799115) (xy 127.99903 69.399115) (xy 129.299821 69.08961) (xy 129.228206 68.121039)
-				(xy 128.130971 68.414774)
+				(xy 125.739667 64.244905) (xy 125.631944 64.345815) (xy 125.532684 64.425672) (xy 125.441785 64.48672)
+				(xy 125.35599 64.533467) (xy 125.181232 64.59972) (xy 125.036344 64.636715) (xy 124.899079 64.671204)
+				(xy 124.748658 64.720228) (xy 124.578483 64.796762) (xy 124.381951 64.913786) (xy 124.827089 65.581747)
+				(xy 125.49505 66.026885) (xy 125.572904 65.901874) (xy 125.633378 65.787906) (xy 125.718607 65.573966)
+				(xy 125.77212 65.372492) (xy 125.813655 65.212341) (xy 125.876819 65.049865) (xy 125.924004 64.963946)
+				(xy 125.985587 64.872872) (xy 126.064564 64.775121) (xy 126.163931 64.669169)
 			)
 		)
